File: cdu-zero.kicad_pcb (KiCad board)
At the start: 4 copper layers, 65 x 30 mm, 5 parts, among them J3 Conn_02x20_Odd_Even

Commit message: Migrated to newer kicad version
Other:
- net class Default removed
